File: hw/kicad/Balloon_bus/Balloon_bus.sch (KiCad schematic (older format))
At the start: 14 parts, among them J1 3V3, J2 DEPLOY SENSOR, J3 SERVO, J4 SOLENOID, J5 LINEAR ACTUATOR, U1 XA1110, U2 MPU-9250-BREAKOUT-R, U3 BMP180-V2, U4 SN754410

Commit message: Moved GPS library to project specific. Additional minor changes in schematic.
Connections:
- wire segments 116 -> 111
Changed lines of the file:
@@
 EESchema Schematic File Version 4
 LIBS:Balloon_bus-cache
-EELAYER 26 0
+EELAYER 29 0
 EELAYER END
 $Descr User 16821 8268
@@
 VBATT
 Wire Wire Line
-	8250 1750 7750 1750
-Wire Wire Line
-	10450 1750 10750 1750
-Wire Wire Line
-	8250 1950 7750 1950
-Wire Wire Line
 	8250 4550 7850 4550
 Text Label 7850 4550 0    70   ~ 0
@@
 U 1 0 6C5DF7BA2912052D
 P 9350 3150
-F 0 "H1H2" V 6650 2050 59  0000 L BNN
+F 0 "H1H2" V 6500 2250 59  0000 L BNN
 F 1 "PC104_CONN" H 9350 3150 50  0001 C CNN
 F 2 "Balloon_bus:PC_104" H 9350 3150 50  0001 C CNN
@@
 GPIO21
 Wire Wire Line
-	15050 5350 15500 5350
-Wire Wire Line
 	12850 5550 12450 5550
 Wire Wire Line
@@
 Wire Wire Line
 	15050 3750 15650 3750
-Wire Wire Line
-	15650 3950 15050 3950
 Text Label 15650 3750 2    70   ~ 0
 MOSI
