File: hw/kicad/DPL/DPL.sch (KiCad schematic (older format))
At the start: 34 parts, among them J0 Programer, J1 DPL1, J2 DPL2, J3 DPL3, J4 DPL4, J5 DPL5, J6 DPL6, J8 BATT, J9 Level shifter, Q1 IRF540N, Q2 IRF540N, Q3 IRF540N, Q4 IRF540N, Q5 IRF540N, Q6 IRF540N, SW1 SW_Reed, SW2 SW_Reed, SW3 SW_Reed, SW4 SW_Reed, SW5 SW_Reed, SW6 SW_Reed, U0 SAMD21E, U1 Payload, Y1 32.768kHz

Commit message: Added level shifter. Increased some drill and pad sizes. Increased power track's thickness.
Parts:
- J9: footprint (none) -> level:Level
Connections:
- net EN_DPL1: no longer U0.7 (PA06/8)
- net EN_DPL2: no longer U0.11 (PA08/4)
- net EN_DPL3: no longer U0.13 (PA10/1)
- net EN_DPL4: no longer U0.15 (PA14/2)
- net LV1: now also U0.7 (PA06/8)
- net LV2: now also U0.11 (PA08/4)
- net LV3: now also U0.13 (PA10/1)
- net LV4: now also U0.15 (PA14/2)
Changed lines of the file:
@@
 	4500 6850 4650 6850
 Text Label 3900 3050 0    50   ~ 0
-EN_DPL1
+LV1
 Text Label 3900 3150 0    50   ~ 0
 DPL_STATUS1
@@
 	3900 3350 4450 3350
 Text Label 3900 3450 0    50   ~ 0
-EN_DPL2
+LV2
 Text Label 3900 3650 0    50   ~ 0
-EN_DPL3
+LV3
 Text Label 3900 3550 0    50   ~ 0
 DPL_STATUS2
@@
 DPL_STATUS3
 Text Label 3900 3850 0    50   ~ 0
-EN_DPL4
+LV4
 Text Label 3900 3950 0    50   ~ 0
 DPL_STATUS4
@@
 	2750 4000 3000 4000
 $Comp
-L power:GND #PWR?
+L power:GND #PWR0113
 U 1 1 5D02A6CC
 P 2800 4150
-F 0 "#PWR?" H 2800 3900 50  0001 C CNN
+F 0 "#PWR0113" H 2800 3900 50  0001 C CNN
 F 1 "GND" H 2805 3977 50  0000 C CNN
 F 2 "" H 2800 4150 50  0001 C CNN
@@
 F 0 "J9" H 2250 7217 50  0000 C CNN
 F 1 "Level shifter" H 2250 7126 50  0000 C CNN
-F 2 "" H 2200 6800 50  0001 C CNN
+F 2 "level:Level" H 2200 6800 50  0001 C CNN
 F 3 "~" H 2200 6800 50  0001 C CNN
 	1    2200 6800
