File: DPL/DPL-A/dpl.sch (KiCad schematic (older format))
At the start: 14 parts, among them J4 D-BUS1, J5 D-BUS2, Q1 PMV16XNR, Q2 PMV16XNR, U3 AV4524, U4 AV4524, U5 DPL

Commit message: New_local_repository
Required
Parts:
- removed D2, D3: LED, Diode_SMD:D_0805_2012Metric_Pad1.15x1.40mm_HandSolder, symbol Device:LED
- removed J4: D-BUS1, Connector_Molex:Molex_PicoBlade_53047-1210_1x12_P1.25mm_Vertical, symbol Connector:Conn_01x12_Male
- removed J5: D-BUS2, Connector_Molex:Molex_PicoBlade_53047-1210_1x12_P1.25mm_Vertical, symbol Connector:Conn_01x12_Male
- removed Q1, Q2: PMV16XNR, Package_TO_SOT_SMD:SOT-23, symbol Transistor_FET:2N7002
- removed R5, R6: 330, Resistor_SMD:R_0603_1608Metric_Pad1.05x0.95mm_HandSolder, symbol Device:R
- removed R7, R8, R9: 1k, Resistor_SMD:R_0603_1608Metric_Pad1.05x0.95mm_HandSolder, symbol Device:R
- removed U3, U4: AV4524, Interrupt:AV4524, symbol Interrupter:AV4524
- removed U5: DPL, Interstage:Type-A, symbol Interstage:DPL
- added Cc1, Cc2: 9pF, Capacitor_SMD:C_0603_1608Metric_Pad1.05x0.95mm_HandSolder, symbol Device:C
- added J2: I2C, Connector_Molex:Molex_PicoBlade_53048-0610_1x06_P1.25mm_Horizontal, symbol Connector:Conn_01x06_Male
- added U1: SAMD21E, Package_QFP:TQFP-32_7x7mm_P0.8mm, symbol Arduino:SAMD21E
- added Y1: 32.768kHz, Crystal:Crystal_SMD_EuroQuartz_EQ161-2Pin_3.2x1.5mm_HandSoldering, symbol Device:Crystal
Connections:
- net labels added: RESET, SCL, SDA, SWCLK, SWDIO, USB_ID, USB_N, USB_P, VDDANA, VDDCORE, VUSB, XIN32, XOUT32
- net labels removed: PORT1, PORT2
- wire segments 64 -> 74
- no-connect marks 4 -> 7
