File: DPL/hw/dpl.sch (KiCad schematic (older format))
At the start: 16 parts, among them J3 Port1, J4 Port2, J5 Port3, J6 Port4, Q1 PMV16XNR, Q2 PMV16XNR, Q3 PMV16XNR, Q4 PMV16XNR

Commit message: New_local_repository
Required
Parts:
- removed J3: Port1, TerminalBlock:TerminalBlock_bornier-3_P5.08mm, symbol Connector:Screw_Terminal_01x03
- removed J4: Port2, TerminalBlock:TerminalBlock_bornier-3_P5.08mm, symbol Connector:Screw_Terminal_01x03
- removed J5: Port3, TerminalBlock:TerminalBlock_bornier-3_P5.08mm, symbol Connector:Screw_Terminal_01x03
- removed J6: Port4, TerminalBlock:TerminalBlock_bornier-3_P5.08mm, symbol Connector:Screw_Terminal_01x03
- removed Q1, Q2, Q3, Q4: PMV16XNR, Package_TO_SOT_SMD:SOT-23, symbol Transistor_FET:2N7002
- removed R10, R12, R6, R8: 1k, Resistor_SMD:R_0603_1608Metric_Pad1.05x0.95mm_HandSolder, symbol Device:R
- removed R11, R5, R7, R9: 330, Resistor_SMD:R_0603_1608Metric_Pad1.05x0.95mm_HandSolder, symbol Device:R
- added Cc1, Cc2: 9pF, Capacitor_SMD:C_0603_1608Metric_Pad1.05x0.95mm_HandSolder, symbol Device:C
- added U0: Payload, Payload:PC104-Standard, symbol Payload:Payload
- added U1: SAMD21E, Package_QFP:TQFP-32_7x7mm_P0.8mm, symbol Arduino:SAMD21E
- added Y1: 32.768kHz, Crystal:Crystal_SMD_EuroQuartz_EQ161-2Pin_3.2x1.5mm_HandSoldering, symbol Device:Crystal
Connections:
- net labels added: RESET, SCL, SDA, SWCLK, SWDIO, USB_ID, USB_N, USB_P, VDDANA, VDDCORE, VIN, VUSB, XIN32, XOUT32
- net labels removed: V_NiCr
- wire segments 47 -> 70
- no-connect marks 0 -> 9
