File: DPL/hw/DPL-A/DPL.sch (KiCad schematic (older format))
At the start: 6 parts, among them J2 I2C, U1 SAMD21E, Y1 32.768kHz

Commit message: Update DPL.sch
Parts:
- removed Cc1, Cc2: 9pF, Capacitor_SMD:C_0603_1608Metric_Pad1.05x0.95mm_HandSolder, symbol Device:C
- removed J2: I2C, Connector_Molex:Molex_PicoBlade_53048-0610_1x06_P1.25mm_Horizontal, symbol Connector:Conn_01x06_Male
- removed R10: 0, Resistor_SMD:R_0603_1608Metric_Pad1.05x0.95mm_HandSolder, symbol Device:R
- removed U1: SAMD21E, Package_QFP:TQFP-32_7x7mm_P0.8mm, symbol Arduino:SAMD21E
- removed Y1: 32.768kHz, Crystal:Crystal_SMD_EuroQuartz_EQ161-2Pin_3.2x1.5mm_HandSoldering, symbol Device:Crystal
- added D2, D3: LED, Diode_SMD:D_0805_2012Metric_Pad1.15x1.40mm_HandSolder, symbol Device:LED
- added J4: D-BUS1, Connector_Molex:Molex_PicoBlade_53047-1210_1x12_P1.25mm_Vertical, symbol Connector:Conn_01x12_Male
- added J5: D-BUS2, Connector_Molex:Molex_PicoBlade_53047-1210_1x12_P1.25mm_Vertical, symbol Connector:Conn_01x12_Male
- added Q1, Q2: PMV16XNR, Package_TO_SOT_SMD:SOT-23, symbol Transistor_FET:2N7002
- added R5, R6: 330, Resistor_SMD:R_0603_1608Metric_Pad1.05x0.95mm_HandSolder, symbol Device:R
- added R7, R8, R9: 1k, Resistor_SMD:R_0603_1608Metric_Pad1.05x0.95mm_HandSolder, symbol Device:R
- added U3, U4: AV4524, Interrupt:AV4524, symbol Interrupter:AV4524
- added U5: DPL, Interstage:Type-A, symbol Interstage:DPL
Connections:
- net labels added: PORT1, PORT2
- net labels removed: RESET, SCL, SDA, SWCLK, SWDIO, USB_ID, USB_N, USB_P, VAUX2, VDDANA, VDDCORE, VUSB, XIN32, XOUT32
- wire segments 76 -> 64
- no-connect marks 7 -> 4

Commit message: Fixed a commit error in which the DPL.sh file was replaced with the dpl.sh file.
Parts:
- removed D2, D3: LED, Diode_SMD:D_0805_2012Metric_Pad1.15x1.40mm_HandSolder, symbol Device:LED
- removed J4: D-BUS1, Connector_Molex:Molex_PicoBlade_53047-1210_1x12_P1.25mm_Vertical, symbol Connector:Conn_01x12_Male
- removed J5: D-BUS2, Connector_Molex:Molex_PicoBlade_53047-1210_1x12_P1.25mm_Vertical, symbol Connector:Conn_01x12_Male
- removed Q1, Q2: PMV16XNR, Package_TO_SOT_SMD:SOT-23, symbol Transistor_FET:2N7002
- removed R5, R6: 330, Resistor_SMD:R_0603_1608Metric_Pad1.05x0.95mm_HandSolder, symbol Device:R
- removed R7, R8, R9: 1k, Resistor_SMD:R_0603_1608Metric_Pad1.05x0.95mm_HandSolder, symbol Device:R
- removed U3, U4: AV4524, Interrupt:AV4524, symbol Interrupter:AV4524
- removed U5: DPL, Interstage:Type-A, symbol Interstage:DPL
- added Cc1, Cc2: 9pF, Capacitor_SMD:C_0603_1608Metric_Pad1.05x0.95mm_HandSolder, symbol Device:C
- added J2: I2C, Connector_Molex:Molex_PicoBlade_53048-0610_1x06_P1.25mm_Horizontal, symbol Connector:Conn_01x06_Male
- added R10: 0, Resistor_SMD:R_0603_1608Metric_Pad1.05x0.95mm_HandSolder, symbol Device:R
- added U1: SAMD21E, Package_QFP:TQFP-32_7x7mm_P0.8mm, symbol Arduino:SAMD21E
- added Y1: 32.768kHz, Crystal:Crystal_SMD_EuroQuartz_EQ161-2Pin_3.2x1.5mm_HandSoldering, symbol Device:Crystal
Connections:
- net labels added: RESET, SCL, SDA, SWCLK, SWDIO, USB_ID, USB_N, USB_P, VAUX2, VDDANA, VDDCORE, VUSB, XIN32, XOUT32
- net labels removed: PORT1, PORT2
- wire segments 64 -> 76
- no-connect marks 4 -> 7
